Commit message: lidarのmoveitでの認識スクリプトを作成途中

File: catkin_ws/src/mycobot_320_moveit/config/gazebo_mycobot_pro.urdf (robot description, URDF)
Before this commit: robot mycobot_pro, 8 links, 7 joints
Links:
- link base_link: geometry collision cylinder length=0.100 radius=0.0725; visual mesh filename=package://mycobot_320_moveit/urdf/320_urdf/base.dae
- link link1: geometry collision cylinder length=0.106 radius=0.043; visual mesh filename=package://mycobot_320_moveit/urdf/320_urdf/link1_1.dae
- link link2: geometry collision cylinder length=0.18 radius=0.036; visual mesh filename=package://mycobot_320_moveit/urdf/320_urdf/link2.dae
- link link3: geometry collision cylinder length=0.14 radius=0.0305; visual mesh filename=package://mycobot_320_moveit/urdf/320_urdf/link3.dae
- link link4: geometry collision cylinder length=0.083 radius=0.029; visual mesh filename=package://mycobot_320_moveit/urdf/320_urdf/link4.dae
- link link5: geometry collision cylinder length=0.0849 radius=0.029; visual mesh filename=package://mycobot_320_moveit/urdf/320_urdf/link5.dae
- link link6: geometry collision cylinder length=0.0225 radius=0.026; visual mesh filename=package://mycobot_320_moveit/urdf/320_urdf/link6.dae

File: catkin_ws/src/mycobot_320_moveit/urdf/k3hand.urdf.xacro (robot description, xacro)
@@ -4,5 +4,5 @@
     <visual>
       <geometry>
-        <mesh filename="package://myrobot/urdf/k3_urdf/wrist.dae" />
+        <mesh filename="package://mycobot_320_moveit/urdf/k3_urdf/wrist.dae" />
       </geometry>
       <origin xyz="0 0 0" rpy="0 0 0" />
@@ -22,5 +22,5 @@
     <visual>
       <geometry>
-        <mesh filename="package://myrobot/urdf/k3_urdf/thumb_met.dae" />
+        <mesh filename="package://mycobot_320_moveit/urdf/k3_urdf/thumb_met.dae" />
       </geometry>
       <origin xyz="0.0 0.0080 0.043" rpy="0 0 0" />
@@ -40,5 +40,5 @@
     <visual>
       <geometry>
-        <mesh filename="package://myrobot/urdf/k3_urdf/thumb_middle_1.dae" />
+        <mesh filename="package://mycobot_320_moveit/urdf/k3_urdf/thumb_middle_1.dae" />
       </geometry>
       <origin xyz="0.0 0.0225 0.0607" />
@@ -58,5 +58,5 @@
     <visual>
       <geometry>
-        <mesh filename="package://myrobot/urdf/k3_urdf/thumb_middle_2.dae" />
+        <mesh filename="package://mycobot_320_moveit/urdf/k3_urdf/thumb_middle_2.dae" />
       </geometry>
       <origin xyz="0.0 0.0225 0.0965" />
@@ -76,5 +76,5 @@
     <visual>
       <geometry>
-        <mesh filename="package://myrobot/urdf/k3_urdf/thumb_tip.dae" />
+        <mesh filename="package://mycobot_320_moveit/urdf/k3_urdf/thumb_tip.dae" />
       </geometry>
       <origin xyz="0.0 0.0225 0.1325" />
@@ -94,5 +94,5 @@
     <visual>
       <geometry>
-        <mesh filename="package://myrobot/urdf/k3_urdf/fing_met_1.dae" />
+        <mesh filename="package://mycobot_320_moveit/urdf/k3_urdf/fing_met_1.dae" />
         <!-- <box size="0.020 0.030 0.012" /> -->
       </geometry>
@@ -113,5 +113,5 @@
     <visual>
       <geometry>
-        <mesh filename="package://myrobot/urdf/k3_urdf/fing_base_1.dae" />
+        <mesh filename="package://mycobot_320_moveit/urdf/k3_urdf/fing_base_1.dae" />
       </geometry>
       <origin xyz="0.015 0.0225 -0.022" />
@@ -131,5 +131,5 @@
     <visual>
       <geometry>
-        <mesh filename="package://myrobot/urdf/k3_urdf/fing_middle_1.dae" />
+        <mesh filename="package://mycobot_320_moveit/urdf/k3_urdf/fing_middle_1.dae" />
       </geometry>
       <origin xyz="0.015 0.0225 -0.022" />
@@ -149,5 +149,5 @@
     <visual>
       <geometry>
-        <mesh filename="package://myrobot/urdf/k3_urdf/fing_tip_1.dae" />
+        <mesh filename="package://mycobot_320_moveit/urdf/k3_urdf/fing_tip_1.dae" />
       </geometry>
       <origin xyz="0.015 0.0225 -0.022" />
@@ -167,5 +167,5 @@
     <visual>
       <geometry>
-        <mesh filename="package://myrobot/urdf/k3_urdf/fing_met_2.dae" />
+        <mesh filename="package://mycobot_320_moveit/urdf/k3_urdf/fing_met_2.dae" />
       </geometry>
       <origin xyz="-0.0225 0.0225 0.00" rpy="0.0 0.0 0.0" />
@@ -185,5 +185,5 @@
     <visual>
       <geometry>
-        <mesh filename="package://myrobot/urdf/k3_urdf/fing_base_2.dae" />
+        <mesh filename="package://mycobot_320_moveit/urdf/k3_urdf/fing_base_2.dae" />
       </geometry>
       <origin xyz="-0.015 0.0225 -0.022" />
@@ -203,5 +203,5 @@
     <visual>
       <geometry>
-        <mesh filename="package://myrobot/urdf/k3_urdf/fing_middle_2.dae" />
+        <mesh filename="package://mycobot_320_moveit/urdf/k3_urdf/fing_middle_2.dae" />
       </geometry>
       <origin xyz="-0.015 0.0225 -0.022" />
@@ -221,5 +221,5 @@
     <visual>
       <geometry>
-        <mesh filename="package://myrobot/urdf/k3_urdf/fing_tip_2.dae" />
+        <mesh filename="package://mycobot_320_moveit/urdf/k3_urdf/fing_tip_2.dae" />
       </geometry>
       <origin xyz="-0.015 0.0225 -0.022" />

File: catkin_ws/src/mycobot_320_moveit/urdf/mycobot_320.urdf.xacro (robot description, xacro)
@@ -28,5 +28,5 @@
     <visual>
       <geometry>
-        <mesh filename="package://myrobot/urdf/320_urdf/link1_1.dae" />
+        <mesh filename="package://mycobot_320_moveit/urdf/320_urdf/link1_1.dae" />
       </geometry>
       <origin xyz="0 0 0 " rpy=" 0 0 0" />
@@ -46,5 +46,5 @@
     <visual>
       <geometry>
-        <mesh filename="package://myrobot/urdf/320_urdf/link2.dae" />
+        <mesh filename="package://mycobot_320_moveit/urdf/320_urdf/link2.dae" />
       </geometry>
       <origin xyz="0 0 0.0587 " rpy=" 0 0 3.1415926" />
@@ -64,5 +64,5 @@
     <visual>
       <geometry>
-        <mesh filename="package://myrobot/urdf/320_urdf/link3.dae" />
+        <mesh filename="package://mycobot_320_moveit/urdf/320_urdf/link3.dae" />
       </geometry>
       <origin xyz="0 0 0.038 " rpy=" 0 0 3.1415926" />
@@ -82,5 +82,5 @@
     <visual>
       <geometry>
-        <mesh filename="package://myrobot/urdf/320_urdf/link4.dae" />
+        <mesh filename="package://mycobot_320_moveit/urdf/320_urdf/link4.dae" />
       </geometry>
       <origin xyz="0 -0.001 0 " rpy=" 0 0 0" />
@@ -100,5 +100,5 @@
     <visual>
       <geometry>
-        <mesh filename="package://myrobot/urdf/320_urdf/link5.dae" />
+        <mesh filename="package://mycobot_320_moveit/urdf/320_urdf/link5.dae" />
       </geometry>
       <origin xyz="0 0.002  0 " rpy=" 0  0 3.1415926" />
@@ -118,5 +118,5 @@
     <visual>
       <geometry>
-        <mesh filename="package://myrobot/urdf/320_urdf/link6.dae" />
+        <mesh filename="package://mycobot_320_moveit/urdf/320_urdf/link6.dae" />
       </geometry>
       <material name="grey">

File: catkin_ws/src/mycobot_320_moveit/urdf/mycobot_k3hand.urdf.xacro (robot description, xacro)
@@ -1,4 +1,4 @@
 <?xml version="1.0"?>
-<robot xmlns:xacro="http://www.ros.org/wiki/xacro" name="myrobot">
+<robot xmlns:xacro="http://www.ros.org/wiki/xacro" name="mycobot_320_moveit">
     <link name="world" />
     <joint name="world2base" type="fixed">
@@ -9,5 +9,5 @@
         <visual>
             <geometry>
-                <mesh filename="package://myrobot/urdf/320_urdf/base.dae" />
+                <mesh filename="package://mycobot_320_moveit/urdf/320_urdf/base.dae" />
             </geometry>
             <origin xyz="0 0 0 " rpy=" 0 0 3.1415926" />
@@ -27,5 +27,5 @@
         <visual>
             <geometry>
-                <mesh filename="package://myrobot/urdf/320_urdf/link1_1.dae" />
+                <mesh filename="package://mycobot_320_moveit/urdf/320_urdf/link1_1.dae" />
             </geometry>
             <origin xyz="0 0 0 " rpy=" 0 0 0" />
@@ -45,5 +45,5 @@
         <visual>
             <geometry>
-                <mesh filename="package://myrobot/urdf/320_urdf/link2.dae" />
+                <mesh filename="package://mycobot_320_moveit/urdf/320_urdf/link2.dae" />
             </geometry>
             <origin xyz="0 0 0.0587 " rpy=" 0 0 3.1415926" />
@@ -63,5 +63,5 @@
         <visual>
             <geometry>
-                <mesh filename="package://myrobot/urdf/320_urdf/link3.dae" />
+                <mesh filename="package://mycobot_320_moveit/urdf/320_urdf/link3.dae" />
             </geometry>
             <origin xyz="0 0 0.038 " rpy=" 0 0 3.1415926" />
@@ -81,5 +81,5 @@
         <visual>
             <geometry>
-                <mesh filename="package://myrobot/urdf/320_urdf/link4.dae" />
+                <mesh filename="package://mycobot_320_moveit/urdf/320_urdf/link4.dae" />
             </geometry>
             <origin xyz="0 -0.001 0 " rpy=" 0 0 0" />
@@ -99,5 +99,5 @@
         <visual>
             <geometry>
-                <mesh filename="package://myrobot/urdf/320_urdf/link5.dae" />
+                <mesh filename="package://mycobot_320_moveit/urdf/320_urdf/link5.dae" />
             </geometry>
             <origin xyz="0 0.002  0 " rpy=" 0  0 3.1415926" />
@@ -117,5 +117,5 @@
         <visual>
             <geometry>
-                <mesh filename="package://myrobot/urdf/320_urdf/link6.dae" />
+                <mesh filename="package://mycobot_320_moveit/urdf/320_urdf/link6.dae" />
             </geometry>
             <material name="grey">
@@ -203,5 +203,5 @@
         </inertial>
     </link>
-    <xacro:include filename="$(find myrobot)/urdf/k3hand.urdf.xacro" />
+    <xacro:include filename="$(find mycobot_320_moveit)/urdf/k3hand.urdf.xacro" />
     <joint name="arm_to_hand" type="fixed">
         <parent link="link6" />

File: catkin_ws/src/mycobot_320_moveit/urdf/mycobot_pro_320_m5_2020.urdf.xacro (robot description, xacro)
@@ -6,5 +6,5 @@
       <geometry>
 	     <!--- 0.0 0 -0.04  1.5708 3.14159-->
-       <mesh filename="package://myrobot/urdf/mycobot_320_m5_2020/base.dae"/>
+       <mesh filename="package://mycobot_320_moveit/urdf/mycobot_320_m5_2020/base.dae"/>
       </geometry>
     <origin xyz = "0.0 0 0 " rpy = " 0 0 3.1415926"/>
@@ -13,5 +13,5 @@
       <geometry>
 	     <!--- 0.0 0 -0.04  1.5708 3.14159-->
-       <mesh filename="package://myrobot/urdf/mycobot_320_m5_2020/base.dae"/>
+       <mesh filename="package://mycobot_320_moveit/urdf/mycobot_320_m5_2020/base.dae"/>
         </geometry>
         <origin xyz = "0.0 0 0 " rpy = " 0 0 3.1415926"/>
@@ -21,5 +21,5 @@
     <visual>
       <geometry>
-       <mesh filename="package://myrobot/urdf/mycobot_320_m5_2020/link1.dae"/>
+       <mesh filename="package://mycobot_320_moveit/urdf/mycobot_320_m5_2020/link1.dae"/>
       </geometry>
     <origin xyz = "0 0 0 " rpy = " 0 0 0"/>
@@ -27,5 +27,5 @@
     <collision>
      <geometry>
-       <mesh filename="package://myrobot/urdf/mycobot_320_m5_2020/link1.dae"/>
+       <mesh filename="package://mycobot_320_moveit/urdf/mycobot_320_m5_2020/link1.dae"/>
       </geometry>
       <origin xyz = "0 0 0 " rpy = " 0 0 0"/>
@@ -35,5 +35,5 @@
     <visual>
       <geometry>
-       <mesh filename="package://myrobot/urdf/mycobot_320_m5_2020/link2.dae"/>
+       <mesh filename="package://mycobot_320_moveit/urdf/mycobot_320_m5_2020/link2.dae"/>
       </geometry>
       <origin xyz = "0 0 0.0587 " rpy = " 0 0 3.1415926"/>
@@ -41,5 +41,5 @@
     <collision>
       <geometry>
-       <mesh filename="package://myrobot/urdf/mycobot_320_m5_2020/link2.dae"/>
+       <mesh filename="package://mycobot_320_moveit/urdf/mycobot_320_m5_2020/link2.dae"/>
       </geometry>
       <origin xyz = "0 0 0.0587 " rpy = " 0 0 3.1415926"/>
@@ -50,5 +50,5 @@
       <geometry>
        <!--- 0.0 0 -0.04 -->
-       <mesh filename="package://myrobot/urdf/mycobot_320_m5_2020/link3.dae"/>
+       <mesh filename="package://mycobot_320_moveit/urdf/mycobot_320_m5_2020/link3.dae"/>
       </geometry>
     <origin xyz = "0 0 0.038 " rpy = " 0 0 3.1415926"/>
@@ -57,5 +57,5 @@
       <geometry>
        <!--- 0.0 0 -0.04 -->
-       <mesh filename="package://myrobot/urdf/mycobot_320_m5_2020/link3.dae"/>
+       <mesh filename="package://mycobot_320_moveit/urdf/mycobot_320_m5_2020/link3.dae"/>
       </geometry>
       <origin xyz = "0 0 0.038 " rpy = " 0 0 3.1415926"/>
@@ -66,5 +66,5 @@
       <geometry>
        <!--- 0.0 0 -0.04 -->
-       <mesh filename="package://myrobot/urdf/mycobot_320_m5_2020/link4.dae"/>
+       <mesh filename="package://mycobot_320_moveit/urdf/mycobot_320_m5_2020/link4.dae"/>
       </geometry>
     <origin xyz = "0 -0.001 0 " rpy = " 0 0 0"/>
@@ -73,5 +73,5 @@
        <geometry>
        <!--- 0.0 0 -0.04 -->
-       <mesh filename="package://myrobot/urdf/mycobot_320_m5_2020/link4.dae"/>
+       <mesh filename="package://mycobot_320_moveit/urdf/mycobot_320_m5_2020/link4.dae"/>
       </geometry>
       <origin xyz = "0 -0.001 0 " rpy = " 0 0 0"/>
@@ -82,5 +82,5 @@
       <geometry>
        <!--- 0.0 0 -0.04 -->
-       <mesh filename="package://myrobot/urdf/mycobot_320_m5_2020/link5.dae"/>
+       <mesh filename="package://mycobot_320_moveit/urdf/mycobot_320_m5_2020/link5.dae"/>
       </geometry>
     <origin xyz = "0 0.002  0 " rpy = " 0  0 3.1415926"/>
@@ -89,5 +89,5 @@
       <geometry>
        <!--- 0.0 0 -0.04 -->
-       <mesh filename="package://myrobot/urdf/mycobot_320_m5_2020/link5.dae"/>
+       <mesh filename="package://mycobot_320_moveit/urdf/mycobot_320_m5_2020/link5.dae"/>
       </geometry>
     <origin xyz = "0 0.002  0 " rpy = " 0  0 3.1415926"/>
@@ -98,5 +98,5 @@
       <geometry>
       <!--- 0.0 0 -0.04 -->
-       <mesh filename="package://myrobot/urdf/mycobot_320_m5_2020/link6.dae"/>
+       <mesh filename="package://mycobot_320_moveit/urdf/mycobot_320_m5_2020/link6.dae"/>
       </geometry>
     <origin xyz = "-0.502 -0.090 -0.096 " rpy = " 0 1.5708 0"/>
@@ -105,5 +105,5 @@
       <geometry>
        <!--- 0.0 0 -0.04 -->
-       <mesh filename="package://myrobot/urdf/mycobot_320_m5_2020/link6.dae"/>
+       <mesh filename="package://mycobot_320_moveit/urdf/mycobot_320_m5_2020/link6.dae"/>
       </geometry>
     <origin xyz = "-0.502 -0.090 -0.096 " rpy = " 0 1.5708 0"/>

File: catkin_ws/src/mycobot_320_moveit/urdf/myrobot.urdf.xacro (robot description, xacro)
@@ -1,4 +1,4 @@
 <?xml version="1.0"?>
-<robot xmlns:xacro="http://www.ros.org/wiki/xacro" name="myrobot">
+<robot xmlns:xacro="http://www.ros.org/wiki/xacro" name="mycobot_320_moveit">
     <link name="world" />
     <joint name="world2base" type="fixed">
@@ -9,5 +9,5 @@
         <visual>
             <geometry>
-                <mesh filename="package://myrobot/urdf/320_urdf/base.dae" />
+                <mesh filename="package://mycobot_320_moveit/urdf/320_urdf/base.dae" />
             </geometry>
             <origin xyz="0 0 0 " rpy=" 0 0 3.1415926" />
@@ -27,5 +27,5 @@
         <visual>
             <geometry>
-                <mesh filename="package://myrobot/urdf/320_urdf/link1_1.dae" />
+                <mesh filename="package://mycobot_320_moveit/urdf/320_urdf/link1_1.dae" />
             </geometry>
             <origin xyz="0 0 0 " rpy=" 0 0 0" />
@@ -45,5 +45,5 @@
         <visual>
             <geometry>
-                <mesh filename="package://myrobot/urdf/320_urdf/link2.dae" />
+                <mesh filename="package://mycobot_320_moveit/urdf/320_urdf/link2.dae" />
             </geometry>
             <origin xyz="0 0 0.0587 " rpy=" 0 0 3.1415926" />
@@ -63,5 +63,5 @@
         <visual>
             <geometry>
-                <mesh filename="package://myrobot/urdf/320_urdf/link3.dae" />
+                <mesh filename="package://mycobot_320_moveit/urdf/320_urdf/link3.dae" />
             </geometry>
             <origin xyz="0 0 0.038 " rpy=" 0 0 3.1415926" />
@@ -81,5 +81,5 @@
         <visual>
             <geometry>
-                <mesh filename="package://myrobot/urdf/320_urdf/link4.dae" />
+                <mesh filename="package://mycobot_320_moveit/urdf/320_urdf/link4.dae" />
             </geometry>
             <origin xyz="0 -0.001 0 " rpy=" 0 0 0" />
@@ -99,5 +99,5 @@
         <visual>
             <geometry>
-                <mesh filename="package://myrobot/urdf/320_urdf/link5.dae" />
+                <mesh filename="package://mycobot_320_moveit/urdf/320_urdf/link5.dae" />
             </geometry>
             <origin xyz="0 0.002  0 " rpy=" 0  0 3.1415926" />
@@ -117,5 +117,5 @@
         <visual>
             <geometry>
-                <mesh filename="package://myrobot/urdf/320_urdf/link6.dae" />
+                <mesh filename="package://mycobot_320_moveit/urdf/320_urdf/link6.dae" />
             </geometry>
             <material name="grey">
