Commit message: 雛形作成

File: catkin_ws/src/core_moveit/config/gazebo_dual_arm_robot.urdf (robot description, URDF)
Before this commit: robot dual_arm_robot, 15 links, 14 joints
Joints:
- joint joint_w: origin xyz=0.5 0 0 rpy=0 0 0 -> xyz=0 0.3 0 rpy=0 0 0

Commit message: make_demo start

File: catkin_ws/src/core_moveit/config/gazebo_dual_arm_robot.urdf (robot description, URDF)
Before this commit: robot dual_arm_robot, 15 links, 14 joints
Joints:
- joint joint_w: origin xyz=0 0.3 0 rpy=0 0 0 -> xyz=0.05 0.45 0 rpy=0 0 0

Commit message: for experiment

File: catkin_ws/src/core_moveit/config/gazebo_dual_arm_robot.urdf (robot description, URDF)
Before this commit: robot dual_arm_robot, 15 links, 14 joints
Joints:
- joint joint_w: origin xyz=0.05 0.45 0 rpy=0 0 0 -> xyz=0.06 0.47 0 rpy=0 0 0
